Commit message: Imu broadcaster specific changes

File: description/urdf/robot_core.xacro (robot description, xacro)
@@ -1,20 +1,18 @@
 <?xml version="1.0"?>
-<robot xmlns:xacro="http://www.ros.org/wiki/xacro">
+<robot name="maus" xmlns:xacro="http://www.ros.org/wiki/xacro">
     <xacro:include filename="inertial_macros.xacro" />
-    <xacro:property name="chassis_length" value="0.335" />
-    <xacro:property name="chassis_width" value="0.265" />
-    <xacro:property name="chassis_height" value="0.138" />
-    <xacro:property name="chassis_mass" value="1.0" />
+    <!-- <xacro:include filename="inertial_macros.xacro" /> -->
+    <xacro:property name="chassis_length" value="0.206" />
+    <xacro:property name="chassis_width" value="0.125" />
+    <xacro:property name="chassis_height" value="0.08" />
+    <xacro:property name="com_to_axis" value="0.028" />
+    <xacro:property name="base_to_imu" value="0.025" />
+    <xacro:property name="wheel_separation" value="0.127" />
+    <xacro:property name="wheel_width" value="0.025" />
     <xacro:property name="wheel_radius" value="0.033" />
-    <xacro:property name="wheel_thickness" value="0.026" />
     <xacro:property name="wheel_mass" value="0.05" />
-    <xacro:property name="wheel_offset_x" value="0.226" />
-    <xacro:property name="wheel_offset_y" value="0.1485" />
-    <xacro:property name="wheel_offset_z" value="0.01" />
-    <xacro:property name="caster_wheel_radius" value="0.01" />
+    <xacro:property name="caster_wheel_radius" value="0.033" />
     <xacro:property name="caster_wheel_mass" value="0.01" />
-    <xacro:property name="caster_wheel_offset_x" value="0.075" />
-    <xacro:property name="caster_wheel_offset_z"
-        value="${wheel_offset_z - wheel_radius + caster_wheel_radius}" />
+    <!-- COLORS -->
     <material name="white">
         <color rgba="1 1 1 1" />
@@ -32,104 +30,61 @@
         <color rgba="1 0 0 1" />
     </material>
-    <!-- BASE LINK -->
+    <!-- LINKS -->
     <link name="base_link">
     </link>
-    <!-- BASE_FOOTPRINT LINK -->
-    <joint name="base_footprint_joint" type="fixed">
-        <parent link="base_link" />
-        <child link="base_footprint" />
-        <origin xyz="0 0 0" rpy="0 0 0" />
-    </joint>
-    <link name="base_footprint">
+    <link name="chassis_link">
+      <visual>
+        <geometry>
+          <box size="${chassis_length} ${chassis_width} ${chassis_height}"/>
+            </geometry>
+            <origin xyz="${com_to_axis} 0 ${chassis_height/2}" rpy="0 0 0" />
+        <collision>
+            <origin xyz="${com_to_axis} 0 ${chassis_height/2}" rpy="0 0 0" />
+            <box size="${chassis_length} ${chassis_width} ${chassis_height}"/>
+            <geometry>
+                <box size="${chassis_length} ${chassis_width} ${chassis_height}"/>
+            </geometry>
+            <xacro:inertial_box mass="0.5" x="${chassis_length}" y="${chassis_width}"
+                z="${chassis_height}">
+                <origin xyz="${com_to_axis} 0 0" rpy="0 0 0" />
+            </xacro:inertial_box>
+        </collision>
+      </visual>
     </link>
-    <!-- CHASSIS LINK -->
-    <joint name="chassis_joint" type="fixed">
-        <parent link="base_link" />
-        <child link="chassis" />
-        <origin xyz="${-wheel_offset_x} 0 ${-wheel_offset_z}" />
-    </joint>
-    <link name="chassis">
-        <visual>
-            <origin xyz="${chassis_length/2} 0 ${chassis_height/2}" />
+    <link name="left_wheel_link">
+      <visual>
             <geometry>
-                <box size="${chassis_length} ${chassis_width} ${chassis_height}" />
-            </geometry>
-            <material name="orange" />
-        </visual>
-        <collision>
-            <origin xyz="${chassis_length/2} 0 ${chassis_height/2}" />
-            <geometry>
-                <box size="${chassis_length} ${chassis_width} ${chassis_height}" />
-            </geometry>
-        </collision>
-        <xacro:inertial_box mass="0.5" x="${chassis_length}" y="${chassis_width}"
-            z="${chassis_height}">
-            <origin xyz="${chassis_length/2} 0 ${chassis_height/2}" rpy="0 0 0" />
-        </xacro:inertial_box>
-    </link>
-    <gazebo reference="chassis">
-        <material>Gazebo/Orange</material>
-    </gazebo>
-    <!-- LEFT WHEEL LINK -->
-    <joint name="left_wheel_joint" type="continuous">
-        <parent link="base_link" />
-        <child link="left_wheel" />
-        <origin xyz="0 ${wheel_offset_y} 0" rpy="-${pi/2} 0 0" />
-        <axis xyz="0 0 1" />
-    </joint>
-    <link name="left_wheel">
-        <visual>
-            <geometry>
-                <cylinder radius="${wheel_radius}" length="${wheel_thickness}" />
+                <cylinder radius="${wheel_radius}" length="${wheel_width}" />
             </geometry>
             <material name="blue" />
-        </visual>
-        <collision>
-            <geometry>
-                <sphere radius="${wheel_radius}" />
-            </geometry>
-        </collision>
-        <xacro:inertial_cylinder mass="${wheel_mass}" length="${wheel_thickness}"
+      </visual>
+      <collision>
+        <geometry>
+                <cylinder radius="${wheel_radius}" length="${wheel_width}" />
+        </geometry>
+      </collision>
+        <xacro:inertial_cylinder mass="${wheel_mass}" length="${wheel_width}"
             radius="${wheel_radius}">
             <origin xyz="0 0 0" rpy="0 0 0" />
         </xacro:inertial_cylinder>
     </link>
-    <gazebo reference="left_wheel">
-        <material>Gazebo/Blue</material>
-    </gazebo>
-    <!-- RIGHT WHEEL LINK -->
-    <joint name="right_wheel_joint" type="continuous">
-        <parent link="base_link" />
-        <child link="right_wheel" />
-        <origin xyz="0 ${-wheel_offset_y} 0" rpy="${pi/2} 0 0" />
-        <axis xyz="0 0 -1" />
-    </joint>
-    <link name="right_wheel">
-        <visual>
+    <link name="right_wheel_link">
+      <visual>
             <geometry>
-                <cylinder radius="${wheel_radius}" length="${wheel_thickness}" />
+                <cylinder radius="${wheel_radius}" length="${wheel_width}" />
             </geometry>
             <material name="blue" />
-        </visual>
-        <collision>
-            <geometry>
-                <sphere radius="${wheel_radius}" />
-            </geometry>
-        </collision>
-        <xacro:inertial_cylinder mass="${wheel_mass}" length="${wheel_thickness}"
+      </visual>
+      <collision>
+        <geometry>
+                <cylinder radius="${wheel_radius}" length="${wheel_width}" />
+        </geometry>
+      </collision>
+        <xacro:inertial_cylinder mass="${wheel_mass}" length="${wheel_width}"
             radius="${wheel_radius}">
             <origin xyz="0 0 0" rpy="0 0 0" />
         </xacro:inertial_cylinder>
     </link>
-    <gazebo reference="right_wheel">
-        <material>Gazebo/Blue</material>
-    </gazebo>
-    <!-- CASTER WHEEL LINK -->
-    <joint name="caster_wheel_joint" type="fixed">
-        <parent link="chassis" />
-        <child link="caster_wheel" />
-        <origin xyz="${caster_wheel_offset_x} 0 ${caster_wheel_offset_z}" />
-    </joint>
-    <link name="caster_wheel">
+    <link name="caster_wheel_link">
         <visual>
             <geometry>
@@ -147,8 +102,33 @@
         </xacro:inertial_sphere>
     </link>
-    <gazebo reference="caster_wheel">
-        <material>Gazebo/White</material>
-        <mu1 value="0.001" />
-        <mu2 value="0.001" />
-    </gazebo>
+    <link name="imu_link">
+    </link>
+<!-- JOINTS -->
+    <joint name="chassis_joint" type="fixed">
+      <parent link="base_link"/>
+      <child link="chassis_link" />
+      <origin xyz="${chassis_length/2 - com_to_axis} 0 0 "/>
+    </joint>
+    <joint name="left_wheel_joint" type="continuous">
+      <parent link="chassis_link" />
+      <child link="left_wheel_link" />
+      <origin xyz="0 ${wheel_separation/2} 0" rpy="-${pi/2} 0 0" />
+      <axis xyz="0 0 1" />
+    </joint>
+    <joint name="right_wheel_joint" type="continuous">
+      <parent link="chassis_link" />
+      <child link="right_wheel_link" />
+      <origin xyz="0 ${-wheel_separation/2} 0" rpy="${pi/2} 0 0" />
+      <axis xyz="0 0 -1" />
+    </joint>
+    <joint name="caster_wheel_joint" type="fixed">
+      <parent link="chassis_link"/>
+      <child link="caster_wheel_link"/>
+      <origin xyz="${chassis_length/2 + com_to_axis - caster_wheel_radius}  0 0" rpy="${pi/2} 0 0" />
+    </joint>
+    <joint name="imu_joint" type="fixed">
+      <parent link="base_link"/>
+      <child link="imu_link"/>
+      <origin xyz="${base_to_imu} 0 0" rpy="${pi/2} 0 0" />
+    </joint>
 </robot>
